File: schematics/shud.kicad_pcb (KiCad board)
At the start: 2 copper layers, 12 parts, among them P1 JTAG, P2 SPI1, U1 STM32F303_K8T6, U2 APE8865N-33-HF-3

Commit message: start writing conclusion
Parts:
- C1, C2, C3: footprint Capacitors_ThroughHole:C_Disc_D3_P2.5 -> Capacitors_ThroughHole:C_Disc_D6_P5
- R1, R2, R3, R4: footprint Resistors_ThroughHole:Resistor_Horizontal_RM10mm -> Resistors_ThroughHole:Resistor_Horizontal_RM7mm
- U2: footprint TO_SOT_Packages_THT:TO-92_Horizontal1_Inline_Narrow_Oval -> TO_SOT_Packages_THT:TO-92_Inline_Wide
- moved C3 46.9 mm to (199.4, 121.9), turned to 180 degrees
- moved BT1 38.1 mm to (181.6, 115.6)
- moved C1 36.7 mm to (199.4, 113.0)
- moved U2 35.9 mm to (185.4, 133.3), turned to 180 degrees
- moved U1 33.1 mm to (210.8, 115.6)
- moved P1 16.9 mm to (238.8, 111.8)
- moved C2 16.5 mm to (222.2, 113.0), turned to 0 degrees
- moved P2 15.6 mm to (215.9, 134.6)
- moved R3 15.4 mm to (232.4, 130.8)
- moved R4 15.4 mm to (232.4, 134.6)
- moved R1 15.4 mm to (232.4, 123.2)
- moved R2 15.4 mm to (232.4, 127.0)
Routing:
- net /JTDO: track 0.00 -> 42.2 mm, vias 0 -> 1
- net /NSS: track 31.1 -> 15.0 mm, vias 1 -> 0
- net +3V3: track 15.1 -> 29.3 mm
- net /SCK: track 29.3 -> 15.3 mm, vias 1 -> 0
- net /MISO: track 28.3 -> 16.0 mm, vias 1 -> 0
- net /JTCK: track 23.2 -> 34.6 mm, vias 0 -> 1
- net /MOSI: track 28.0 -> 16.7 mm, vias 1 -> 0
- net /JNTRST: track 24.7 -> 32.2 mm, vias 0 -> 1
- net /JTMS: track 18.9 -> 26.1 mm, vias 2 -> 1
- net /JTDI: track 22.7 -> 29.4 mm, vias 0 -> 1
- net Net-(BT1-Pad1): track 12.3 -> 18.3 mm
- net Net-(P1-Pad17): track 6.15 -> 6.88 mm
- net Net-(P1-Pad15): track 6.67 -> 7.40 mm
- net Net-(P1-Pad11): track 6.15 -> 6.88 mm
- net Net-(P1-Pad19): track 5.62 -> 6.35 mm
- removed copper zone on F.Cu, net +3V3
- removed copper zone on B.Cu, net GND
Other:
- net class Default: trace_width 0.25 -> 0.5; via_dia 1 -> 1.7272; via_drill 0.8 -> 1.016
- rule pad_to_mask_clearance: 0.2 -> 0
